Commit message: feat(description): visual-only industrial robot body
appearance.xacro adds visuals to the existing links only: graphite skirt,
yellow body and deck, counterweight with rounded corners, rubber bumpers,
LED strip, electronics tower with LiDAR, amber beacon, e-stop, front safety
scanners, wheel hubs and a lift cylinder. All sizes in forklift_params.yaml
(appearance); every part is behind the camera optical centres (x = 0.10).
- links, joints, inertials, collisions and gazebo blocks unchanged (57/57)
- robot camera images unchanged (difference = render noise)
- hazard stripe and side label are textured OBJ decals generated at build
  time (sdformat drops URDF visual names, so per-visual materials cannot be
  set); package.xml exports gazebo_model_path ${prefix}/.. for model://
- dark colours compensate for sdformat's x1.25 URDF colour scale
Recorded as DECISIONS D-54.

Co-Authored-By: Claude Opus 5.5 <noreply@anthropic.com>

File: src/forklift_description/urdf/common/materials.xacro (robot description, xacro)
@@ -3,12 +3,26 @@
   materials.xacro
   Görsel renkler (yalnızca <visual>). Fiziksel parametre içermez.
+  gz'de görünen renk: sdformat URDF rengini 1.25 ile çarpar (ölçüldü) ve
+  ogre2 doğrusal → sRGB çevirir; koyu tonlar bu yüzden düşük değerlerle
+  verilir (D-54). RViz bu rengi olduğu gibi gösterir (daha koyu görünür).
   Not: Robotun kameraların görebileceği parçaları (çatallar, taşıyıcı) koli
   mühür renklerinden (kırmızı / yeşil / mavi) bilinçli olarak uzak tutuldu.
+  Görünüm parçaları (components/appearance.xacro) kameraların gerisindedir;
+  acil stop kırmızısı bu yüzden robotun kendi görüntüsüne girmez.
 -->
 <robot xmlns:xacro="http://www.ros.org/wiki/xacro">
-  <material name="forklift_yellow"><color rgba="0.95 0.72 0.08 1.0"/></material>
-  <material name="forklift_dark_grey"><color rgba="0.20 0.20 0.22 1.0"/></material>
+  <material name="forklift_yellow"><color rgba="0.78 0.45 0.02 1.0"/></material>
+  <material name="forklift_dark_grey"><color rgba="0.08 0.08 0.09 1.0"/></material>
   <material name="forklift_steel"><color rgba="0.55 0.56 0.60 1.0"/></material>
   <material name="forklift_rubber"><color rgba="0.05 0.05 0.05 1.0"/></material>
   <material name="forklift_camera"><color rgba="0.10 0.10 0.12 1.0"/></material>
+  <!-- görünüm (appearance.xacro) -->
+  <material name="forklift_graphite"><color rgba="0.035 0.037 0.042 1.0"/></material>
+  <material name="forklift_counterweight"><color rgba="0.06 0.062 0.068 1.0"/></material>
+  <material name="forklift_black"><color rgba="0.012 0.012 0.014 1.0"/></material>
+  <material name="forklift_glass"><color rgba="0.01 0.015 0.025 1.0"/></material>
+  <material name="forklift_chrome"><color rgba="0.45 0.46 0.48 1.0"/></material>
+  <material name="forklift_led"><color rgba="0.85 0.92 0.95 1.0"/></material>
+  <material name="forklift_amber"><color rgba="0.80 0.36 0.0 1.0"/></material>
+  <material name="forklift_estop_red"><color rgba="0.62 0.02 0.02 1.0"/></material>
 </robot>

File: src/forklift_description/urdf/components/chassis.xacro (robot description, xacro)
@@ -6,5 +6,6 @@
                       link ataleti desteklemez).
       base_link     : tahrik aksı merkezi, kütlesiz çerçeve link'i.
-  - chassis: şasi kutusu (chassis_link), base_link'e sabit.
+  - chassis: şasi kutusu (chassis_link), base_link'e sabit. Görünümü
+    components/appearance.xacro → chassis_visuals verir (D-54).
   Not: <collision> elemanları bilinçli olarak adsızdır (DECISIONS D-03).
 -->
@@ -23,9 +24,6 @@
     <xacro:property name="ch" value="${cfg.chassis}"/>
     <link name="${prefix}chassis_link">
-      <visual>
-        <origin xyz="0 0 0" rpy="0 0 0"/>
-        <geometry><box size="${ch.size.x} ${ch.size.y} ${ch.size.z}"/></geometry>
-        <material name="forklift_yellow"/>
-      </visual>
+      <!-- görünüm: appearance.xacro (yalnız visual; collision ve atalet bu kutudur) -->
+      <xacro:chassis_visuals cfg="${cfg}"/>
       <collision>
         <origin xyz="0 0 0" rpy="0 0 0"/>

File: src/forklift_description/urdf/components/drive_wheel.xacro (robot description, xacro)
@@ -20,4 +20,6 @@
         <material name="forklift_rubber"/>
       </visual>
+      <!-- görünüm: sarı göbek (yalnız visual, D-54) -->
+      <xacro:wheel_hub_visual cfg="${cfg}"/>
       <!-- collision_shape: cylinder (spesifikasyon) | sphere (tek nokta temas;
            DECISIONS D-20). Görsel ve atalet her durumda silindirdir. -->

File: src/forklift_description/urdf/components/mast.xacro (robot description, xacro)
@@ -52,4 +52,6 @@
         <geometry><box size="${bar.x} ${bar.y} ${bar.z}"/></geometry>
       </collision>
+      <!-- görünüm: direğin arkasında kaldırma silindiri (yalnız visual, D-54) -->
+      <xacro:lift_cylinder_visual cfg="${cfg}"/>
       <xacro:composite_box_inertial boxes="${[
           dict(m=m_up,  size=[up.x, up.y, up.z],    xyz=[0.0,  ms.upright.y, up_z]),

File: src/forklift_description/urdf/forklift.urdf.xacro (robot description, xacro)
@@ -27,4 +27,5 @@
   <xacro:include filename="components/fork_carriage.xacro"/>
   <xacro:include filename="components/camera.xacro"/>
+  <xacro:include filename="components/appearance.xacro"/>
   <!-- gövde ve yürüyüş -->
   <xacro:forklift_base_frames prefix="${prefix}" cfg="${cfg}"/>
