Commit message: feat(gazebo): factory world and industrial station look
- factory.sdf generated at build time from config/factory.yaml: Open
  Robotics Depot hall (Fuel, pinned) rotated so the source station faces a
  plain door wall; Depot floor collision and its fan_light point lights
  (attenuation 0/0/0, saturated or blackened our models per camera) removed
  via experimental:params; optional clutter: clean
- lights calibrated so the front camera sees the seals within +-6 % of
  station_test; hazard-taped cell, guide lanes with stop bars
  (factory_lanes.yaml ground truth), walkway, pillar guards, signs, props
- stations and parcels: tread plate with colour band, aluminium back plate
  and frame, signs, bay labels, label plates behind the markers, rubber
  ledges, kraft parcels with tape and label; collisions, inertia, frames and
  marker poses byte-identical, seal unchanged
- CC0 ambientCG textures committed; signs/labels generated at build time
- station_sim.launch.py station_world:=station_test|factory, sim.launch.py
  gui_config, bringup world:=factory, factory_gui.config opening camera
- measure_sim_performance.py: RTF, camera rate, CPU/RAM, GPU per world
Recorded as DECISIONS D-53.

Co-Authored-By: Claude Opus 5.5 <noreply@anthropic.com>

File: src/forklift_gazebo/xacro/common.sdf.xacro (robot description, xacro)
@@ -5,5 +5,8 @@
     ambient = ambient_scale · diffuse, specular / roughness / metalness
     station_params.yaml → material'dan. İsteğe bağlı albedo_map (PBR doku).
+  - finish_material: PBR yüzey (station_params.yaml → finishes): albedo,
+    normal ve roughness haritaları model://factory_materials altından.
   - box_inertial: dolu kutu ataleti (SDF), kütle ve kenarlardan hesaplanır.
+  - box_part: collision + visual kutu; box_visual: yalnız visual kutu.
   Çağıran dosya P (station_params.yaml içeriği) özelliğini tanımlamış olmalı.
 -->
@@ -12,4 +15,7 @@
        (share/forklift_gazebo/models/aruco_markers/materials/textures). -->
   <xacro:property name="texture_uri_root" value="model://aruco_markers/materials/textures"/>
+  <!-- CC0 fotoğraf dokuları (depoda) ve build'de üretilen tabela dokuları -->
+  <xacro:property name="finish_uri_root" value="model://factory_materials/materials/textures"/>
+  <xacro:property name="sign_uri_root" value="model://factory_signs/materials/textures"/>
   <xacro:macro name="matte_material" params="rgba albedo_map:=''">
     <xacro:property name="k" value="${P['material']['ambient_scale']}"/>
@@ -30,4 +36,24 @@
     </material>
   </xacro:macro>
+  <!-- PBR yüzey; f = finishes kaydı. rgba albedo ile çarpılır, ambient
+       matte_material'daki gibi ambient_scale · rgba. -->
+  <xacro:macro name="finish_material" params="f">
+    <xacro:property name="k" value="${P['material']['ambient_scale']}"/>
+    <xacro:property name="c" value="${f['rgba']}"/>
+    <xacro:property name="t" value="${finish_uri_root + '/' + f['maps']}"/>
+    <material>
+      <ambient>${round(c[0] * k, 6)} ${round(c[1] * k, 6)} ${round(c[2] * k, 6)} ${c[3]}</ambient>
+      <diffuse>${c[0]} ${c[1]} ${c[2]} ${c[3]}</diffuse>
+      <specular>0.1 0.1 0.1 1</specular>
+      <pbr>
+        <metal>
+          <albedo_map>${t}_albedo.jpg</albedo_map>
+          <normal_map>${t}_normal.jpg</normal_map>
+          <roughness_map>${t}_roughness.jpg</roughness_map>
+          <metalness>${f['metalness']}</metalness>
+        </metal>
+      </pbr>
+    </material>
+  </xacro:macro>
   <!-- Dolu kutu; x, y, z kenar uzunlukları. Tensör link eksenlerinde, kütle
        merkezi link orijininde. -->
@@ -43,7 +69,9 @@
   </xacro:macro>
   <!-- Eksenlere hizalı kutu: collision (isteğe bağlı sürtünmeyle) + visual.
-       mu boşsa <surface> yazılmaz (SDF varsayılanı). Konum ve boyutlar 1 nm'ye
+       mu boşsa <surface> yazılmaz (SDF varsayılanı). finish verilirse visual
+       PBR yüzey kullanır, yoksa rgba mat malzeme. visual_dx: visual'ın x
+       kayması (yalnız görünüm; collision yerinde kalır). Konum ve boyutlar 1 nm'ye
        yuvarlanır: kayan nokta artığı (0.8999999999999999) SDF'te görünmesin. -->
-  <xacro:macro name="box_part" params="name size xyz rgba collision:=true mu:=''">
+  <xacro:macro name="box_part" params="name size xyz rgba collision:=true mu:='' finish:='' visual_dx:=0">
     <xacro:property name="pose_str" value="${round(xyz[0], 9)} ${round(xyz[1], 9)} ${round(xyz[2], 9)} 0 0 0"/>
     <xacro:property name="size_str" value="${round(size[0], 9)} ${round(size[1], 9)} ${round(size[2], 9)}"/>
@@ -57,8 +85,20 @@
       </collision>
     </xacro:if>
-    <visual name="${name}_visual">
-      <pose>${pose_str}</pose>
-      <geometry><box><size>${size_str}</size></box></geometry>
-      <xacro:matte_material rgba="${rgba}"/>
+    <xacro:box_visual name="${name}_visual" size="${size}" xyz="${[xyz[0] + visual_dx, xyz[1], xyz[2]]}"
+                      rgba="${rgba}" finish="${finish}"/>
+  </xacro:macro>
+  <!-- Yalnız visual kutu. Malzeme önceliği: finish → albedo_map → rgba.
+       cast_shadows false: ince süs parçaları (bant, etiket) gölge düşürmesin. -->
+  <xacro:macro name="box_visual" params="name size xyz rgba:='' finish:='' albedo_map:='' cast_shadows:=true">
+    <visual name="${name}">
+      <pose>${round(xyz[0], 9)} ${round(xyz[1], 9)} ${round(xyz[2], 9)} 0 0 0</pose>
+      <geometry><box><size>${round(size[0], 9)} ${round(size[1], 9)} ${round(size[2], 9)}</size></box></geometry>
+      <xacro:unless value="${cast_shadows}"><cast_shadows>false</cast_shadows></xacro:unless>
+      <xacro:if value="${finish != ''}">
+        <xacro:finish_material f="${finish}"/>
+      </xacro:if>
+      <xacro:if value="${finish == ''}">
+        <xacro:matte_material rgba="${rgba if rgba != '' else [1.0, 1.0, 1.0, 1.0]}" albedo_map="${albedo_map}"/>
+      </xacro:if>
     </visual>
   </xacro:macro>

File: src/forklift_gazebo/xacro/parcel.sdf.xacro (robot description, xacro)
@@ -9,4 +9,7 @@
   bakar). Mühür bu yüzde ortalanmış, ayrı visual, collision'ı yok; iç yüzü koli
   yüzüyle aynı hizada, thickness kadar dışarı taşar.
+  Görünüm (yalnız visual, appearance.parcel): oluklu karton gövde, üst yüzde
+  x boyunca koli bandı (+x yüzünden aşağı iner; -x yüzü yalnız mühür içindir),
+  +y yüzünde gönderi etiketi (parcel_label.png).
   Atalet dolu kutu formülüyle hesaplanır. Sürtünme μ = parcel.mu; DART
   min(μA, μB) birleştirir (D-15): koli–çatal 0.8, koli–çıkıntı 0.8.
@@ -27,9 +30,19 @@
   <xacro:property name="sz" value="${B['size']['z']}"/>
   <xacro:property name="seal" value="${B['seal']}"/>
+  <xacro:property name="V" value="${P['appearance']['parcel']}"/>
+  <xacro:property name="deco" value="0.0005"/>  <!-- süs parçalarının yüzeyden taşması -->
   <model name="$(arg name)">
     <link name="parcel_link">
       <xacro:box_inertial mass="${B['mass']}" x="${sx}" y="${sy}" z="${sz}"/>
       <xacro:box_part name="body" size="${[sx, sy, sz]}" xyz="${[0, 0, 0]}"
-                      rgba="${P['colors']['parcel_body']}" mu="${B['mu']}"/>
+                      rgba="${P['colors']['parcel_body']}" mu="${B['mu']}" finish="${P['finishes']['cardboard']}"/>
+      <xacro:box_visual name="tape_top" size="${[sx, V['tape_width'], deco]}" xyz="${[0, 0, sz / 2.0 + deco / 2.0]}"
+                        rgba="${P['colors']['tape']}" cast_shadows="false"/>
+      <xacro:box_visual name="tape_back" size="${[deco, V['tape_width'], V['tape_drop']]}"
+                        xyz="${[sx / 2.0 + deco / 2.0, 0, sz / 2.0 - V['tape_drop'] / 2.0]}"
+                        rgba="${P['colors']['tape']}" cast_shadows="false"/>
+      <xacro:box_visual name="shipping_label" size="${[V['label']['x'], deco, V['label']['z']]}"
+                        xyz="${[0, sy / 2.0 + deco / 2.0, 0]}" cast_shadows="false"
+                        albedo_map="${sign_uri_root}/parcel_label.png"/>
       <xacro:box_part name="seal" collision="false"
                       size="${[seal['thickness'], seal['size']['y'], seal['size']['z']]}"

File: src/forklift_gazebo/xacro/station.sdf.xacro (robot description, xacro)
@@ -18,4 +18,10 @@
     arka plaka     x ∈ [ledge_depth, ledge_depth + back_plate_thickness], z ∈ [0, back_plate_height]
     işaretler      arka plakanın ön yüzünde, standoff kadar önde, yalnız visual
+  Görünüm (yalnız visual, station_params.yaml → appearance, finishes):
+    zemin plakası gözyaşı sac; üstünde istasyon renginde çevre bandı
+    arka plaka alüminyum, visual'ı back_plate_recess kadar geride; işaretlerin
+    arkasında beyaz etiket plakası (işaret ile arka plaka arasında)
+    çıkıntılar kauçuk; arka plakanın arkasında profil çerçeve, üstünde tabela
+    (sign_<renk>.png) ve her bölmede numara etiketi (bay_<k>.png)
 -->
 <sdf version="1.11" xmlns:xacro="http://www.ros.org/wiki/xacro">
@@ -61,4 +67,13 @@
   <xacro:property name="tex_scale" value="${(6 + 2 * M['quiet_zone_cells']) / 6.0}"/>
   <xacro:property name="dict_tag" value="${M['dictionary'].lower().replace('dict_', '')}"/>
+  <!-- görünüm -->
+  <xacro:property name="V" value="${P['appearance']}"/>
+  <xacro:property name="F" value="${P['finishes']}"/>
+  <xacro:property name="band_rgba" value="${C['band_neutral'] if color == 'neutral' else C[color]}"/>
+  <xacro:property name="recess" value="${V['back_plate_recess']}"/>
+  <xacro:property name="pr" value="${V['frame']['profile']}"/>
+  <xacro:property name="fh" value="${V['frame']['height']}"/>
+  <xacro:property name="sign_w" value="${min(V['sign']['width'], W - 2 * pr)}"/>
+  <xacro:property name="sign_h" value="${sign_w / V['sign']['aspect']}"/>
   <!-- Çıkıntı j (0 … N): kanal j-1 ile kanal j arasındaki her şey; uçlarda
        istasyon kenarına kadar. Özyinelemeli makro (xacro'da döngü yok). -->
@@ -68,5 +83,5 @@
     <xacro:box_part name="ledge_${j}" size="${[D, y_hi - y_lo, lh]}"
                     xyz="${[D / 2.0, (y_lo + y_hi) / 2.0, lh / 2.0]}"
-                    rgba="${C['ledge']}" mu="${S['ledge_mu']}"/>
+                    rgba="${C['ledge']}" mu="${S['ledge_mu']}" finish="${F['rubber']}"/>
     <xacro:if value="${j &lt; N}">
       <xacro:ledges j="${j + 1}"/>
@@ -83,4 +98,12 @@
           albedo_map="${texture_uri_root}/aruco_${dict_tag}_id${'%02d' % marker_id}.png"/>
     </visual>
+    <!-- beyaz etiket plakası: ön yüzü işaretin arka yüzü ile arka plaka visual'ı
+         arasında; alt kenarı zemin plakasının üstünde kalır -->
+    <xacro:property name="lm" value="${V['label_margin'][kind]}"/>
+    <xacro:property name="lt" value="${V['label_thickness']}"/>
+    <xacro:property name="lz_lo" value="${max(M[kind]['center_z'] - edge / 2.0 - lm, bt + V['band_height'])}"/>
+    <xacro:property name="lz_hi" value="${M[kind]['center_z'] + edge / 2.0 + lm}"/>
+    <xacro:box_visual name="label_${kind}_${marker_id}" size="${[lt, edge + 2 * lm, lz_hi - lz_lo]}"
+                      xyz="${[D + recess / 2.0, y, (lz_lo + lz_hi) / 2.0]}" rgba="${C['label']}" cast_shadows="false"/>
   </xacro:macro>
   <!-- Bölme i: çerçeve + üst ve alt işaret -->
@@ -89,4 +112,7 @@
     <xacro:marker kind="upper" marker_id="${ids[i]}" y="${y}"/>
     <xacro:marker kind="lower" marker_id="${ids[i] + M['lower_id_offset']}" y="${y}"/>
+    <xacro:box_visual name="bay_label_${ids[i]}" size="${[V['label_thickness'], V['bay_label']['size'], V['bay_label']['size']]}"
+                      xyz="${[D + recess / 2.0, y, V['bay_label']['center_z']]}" cast_shadows="false"
+                      albedo_map="${sign_uri_root}/bay_${'%02d' % ids[i]}.png"/>
     <xacro:if value="${i + 1 &lt; N}">
       <xacro:bays i="${i + 1}"/>
@@ -105,7 +131,27 @@
     <link name="station_link">
       <xacro:box_part name="base_plate" size="${[A + D + T, W, bt]}"
-                      xyz="${[(D + T - A) / 2.0, 0, bt / 2.0]}" rgba="${C[color]}"/>
+                      xyz="${[(D + T - A) / 2.0, 0, bt / 2.0]}" rgba="${C[color]}" finish="${F['tread_plate']}"/>
       <xacro:box_part name="back_plate" size="${[T, W, S['back_plate_height']]}"
-                      xyz="${[D + T / 2.0, 0, S['back_plate_height'] / 2.0]}" rgba="${C['back_plate']}"/>
+                      xyz="${[D + T / 2.0, 0, S['back_plate_height'] / 2.0]}" rgba="${C['back_plate']}"
+                      finish="${F['aluminium']}" visual_dx="${recess}"/>
+      <!-- renk bandı: zemin plakasının üst yüzünde, çevre boyunca -->
+      <xacro:property name="bw" value="${V['band_width']}"/>
+      <xacro:property name="bz" value="${bt + V['band_height'] / 2.0}"/>
+      <xacro:property name="bl" value="${A + D + T}"/>
+      <xacro:box_visual name="band_front" size="${[bw, W, V['band_height']]}" xyz="${[-A + bw / 2.0, 0, bz]}"
+                        rgba="${band_rgba}" cast_shadows="false"/>
+      <xacro:box_visual name="band_left" size="${[bl - bw, bw, V['band_height']]}" xyz="${[(D + T - A + bw) / 2.0, W / 2.0 - bw / 2.0, bz]}"
+                        rgba="${band_rgba}" cast_shadows="false"/>
+      <xacro:box_visual name="band_right" size="${[bl - bw, bw, V['band_height']]}" xyz="${[(D + T - A + bw) / 2.0, -W / 2.0 + bw / 2.0, bz]}"
+                        rgba="${band_rgba}" cast_shadows="false"/>
+      <!-- profil çerçeve: iki dikme + üst kiriş, arka plakanın arkasında -->
+      <xacro:property name="fx" value="${D + T + recess + pr / 2.0}"/>
+      <xacro:box_visual name="frame_post_left" size="${[pr, pr, fh]}" xyz="${[fx, W / 2.0 - pr / 2.0, fh / 2.0]}" finish="${F['aluminium']}"/>
+      <xacro:box_visual name="frame_post_right" size="${[pr, pr, fh]}" xyz="${[fx, -W / 2.0 + pr / 2.0, fh / 2.0]}" finish="${F['aluminium']}"/>
+      <xacro:box_visual name="frame_top" size="${[pr, W - 2 * pr, pr]}" xyz="${[fx, 0, fh - pr / 2.0]}" finish="${F['aluminium']}"/>
+      <!-- tabela: çerçevenin ön yüzüne asılı -->
+      <xacro:box_visual name="sign" size="${[V['sign']['thickness'], sign_w, sign_h]}"
+                        xyz="${[fx - pr / 2.0 - V['sign']['thickness'] / 2.0, 0, V['sign']['top_z'] - sign_h / 2.0]}"
+                        albedo_map="${sign_uri_root}/sign_${color}.png"/>
       <xacro:ledges j="0"/>
       <xacro:bays i="0"/>

Commit message: feat(gazebo): remove ArUco markers; bay lanes and station-coloured floor lanes
Owner decision (D-56): station identity comes from the colour-coded sign,
the bay index from the order of the bullseye pairs, parcel presence from
object detection; the robot must not use surveyed world poses
(markers.yaml stays ground truth only).
- removed upper/lower markers, label plates, ID scheme, ArUco textures,
  detector parameters and tests S4/S5 (shown as KALDIRILDI)
- generate_aruco_textures.py -> generate_station_textures.py,
  model://aruco_markers -> model://station_targets
- bay lane: 40 mm line along every bay axis on the tread plate, station
  colour (yellow at the source); markers.yaml bay_lines; S2 checks
- factory floor lanes in each station's colour, 0.12 m start gap at the hub
- S1/S2 pass (1231 checks); S3, S6, S7, S8 pass; README/ARCHITECTURE/
  DECISIONS/REPORT notes and all station screenshots refreshed

Co-Authored-By: Claude Opus 5.5 <noreply@anthropic.com>

File: src/forklift_gazebo/xacro/common.sdf.xacro (robot description, xacro)
@@ -13,6 +13,6 @@
 <sdf xmlns:xacro="http://www.ros.org/wiki/xacro">
   <!-- Dokuların model:// kökü. CMakeLists.txt aynı dizine kurar
-       (share/forklift_gazebo/models/aruco_markers/materials/textures). -->
-  <xacro:property name="texture_uri_root" value="model://aruco_markers/materials/textures"/>
+       (share/forklift_gazebo/models/station_targets/materials/textures). -->
+  <xacro:property name="texture_uri_root" value="model://station_targets/materials/textures"/>
   <!-- CC0 fotoğraf dokuları (depoda) ve build'de üretilen tabela dokuları -->
   <xacro:property name="finish_uri_root" value="model://factory_materials/materials/textures"/>

File: src/forklift_gazebo/xacro/station.sdf.xacro (robot description, xacro)
@@ -6,6 +6,5 @@
     bays        : bölme sayısı N (≥ 1)
     color       : zemin plakası rengi: red | green | blue | neutral
-    bay_ids     : bölme numaraları k, virgülle ("3,4,5"); boş → 0 … N-1.
-                  Üst işaret ID = k, alt işaret ID = k + lower_id_offset (D-45)
+    bay_ids     : bölme numaraları k, virgülle ("3,4,5"); boş → 0 … N-1 (bölme etiketleri)
     params_file : station_params.yaml (tüm ölçüler buradan; D-02 kuralı)
   Model çerçevesi = station çerçevesi: orijin zeminde, ön kenarın ortasında;
@@ -17,11 +16,12 @@
     çıkıntılar     kanallar arası, x ∈ [0, ledge_depth], z ∈ [0, ledge_height], μ = ledge_mu
     arka plaka     x ∈ [ledge_depth, ledge_depth + back_plate_thickness], z ∈ [0, back_plate_height]
-    işaretler      arka plakanın ön yüzünde, standoff kadar önde, yalnız visual
     hizalama       bölme başına 2 hedef (markers.align.pattern), çıkıntıların ön yüzünde kanalın
                    iki yanında, standoff kadar önde, yalnız visual (D-55)
+    bölme şeridi   zemin plakası üstünde bölme ekseninde, önlük bandından kanal girişine;
+                   istasyon renginde (kaynakta sarı), yalnız visual (D-56)
+  ArUco işaretleri D-56 ile kaldırıldı.
   Görünüm (yalnız visual, station_params.yaml → appearance, finishes):
     zemin plakası gözyaşı sac; üstünde istasyon renginde çevre bandı
-    arka plaka alüminyum, visual'ı back_plate_recess kadar geride; işaretlerin
-    arkasında beyaz etiket plakası (işaret ile arka plaka arasında)
+    arka plaka alüminyum, visual'ı back_plate_recess kadar geride
     çıkıntılar kauçuk; arka plakanın arkasında profil çerçeve, üstünde tabela
     (sign_<renk>.png) ve her bölmede numara etiketi (bay_<k>.png)
@@ -64,13 +64,9 @@
   <xacro:property name="A" value="${S['apron_depth']}"/>
   <xacro:property name="bt" value="${S['base_plate_thickness']}"/>
-  <!-- işaret kutusu merkezi x: ön yüzü D - standoff - thickness -->
-  <xacro:property name="marker_cx" value="${D - M['standoff'] - M['thickness'] / 2.0}"/>
-  <!-- doku kenarı = siyah kare · (6 + 2 · beyaz kenar hücresi) / 6 -->
-  <xacro:property name="tex_scale" value="${(6 + 2 * M['quiet_zone_cells']) / 6.0}"/>
-  <xacro:property name="dict_tag" value="${M['dictionary'].lower().replace('dict_', '')}"/>
   <!-- görünüm -->
   <xacro:property name="V" value="${P['appearance']}"/>
   <xacro:property name="F" value="${P['finishes']}"/>
   <xacro:property name="band_rgba" value="${C['band_neutral'] if color == 'neutral' else C[color]}"/>
+  <xacro:property name="lane_rgba" value="${C['lane_neutral'] if color == 'neutral' else C[color]}"/>
   <xacro:property name="recess" value="${V['back_plate_recess']}"/>
   <xacro:property name="pr" value="${V['frame']['profile']}"/>
@@ -90,23 +86,4 @@
     </xacro:if>
   </xacro:macro>
-  <!-- İşaret: 1 mm kutu, dokulu ön yüz -x'e bakar; collision yok. Kutunun
-       -x yüzünde doku ayna görüntüsü olmadan okunur (Faz 1 sondası, D-47). -->
-  <xacro:macro name="marker" params="kind marker_id y">
-    <xacro:property name="edge" value="${M[kind]['size'] * tex_scale}"/>
-    <visual name="marker_${kind}_${marker_id}">
-      <pose>${round(marker_cx, 9)} ${round(y, 9)} ${M[kind]['center_z']} 0 0 0</pose>
-      <geometry><box><size>${M['thickness']} ${round(edge, 9)} ${round(edge, 9)}</size></box></geometry>
-      <xacro:matte_material rgba="${C['marker']}"
-          albedo_map="${texture_uri_root}/aruco_${dict_tag}_id${'%02d' % marker_id}.png"/>
-    </visual>
-    <!-- beyaz etiket plakası: ön yüzü işaretin arka yüzü ile arka plaka visual'ı
-         arasında; alt kenarı zemin plakasının üstünde kalır -->
-    <xacro:property name="lm" value="${V['label_margin'][kind]}"/>
-    <xacro:property name="lt" value="${V['label_thickness']}"/>
-    <xacro:property name="lz_lo" value="${max(M[kind]['center_z'] - edge / 2.0 - lm, bt + V['band_height'])}"/>
-    <xacro:property name="lz_hi" value="${M[kind]['center_z'] + edge / 2.0 + lm}"/>
-    <xacro:box_visual name="label_${kind}_${marker_id}" size="${[lt, edge + 2 * lm, lz_hi - lz_lo]}"
-                      xyz="${[D + recess / 2.0, y, (lz_lo + lz_hi) / 2.0]}" rgba="${C['label']}" cast_shadows="false"/>
-  </xacro:macro>
   <!-- Hizalama hedefi: kanal kenarına edge_gap kadar uzakta, çıkıntı ön yüzünün
        ortasında; dokulu yüz -x'e bakar. station_layout.align_points ile aynı formül. -->
@@ -118,9 +95,12 @@
                       albedo_map="${texture_uri_root}/align_${AL['pattern']}.png"/>
   </xacro:macro>
-  <!-- Bölme i: çerçeve + üst ve alt işaret + iki hizalama hedefi -->
+  <!-- Bölme i: iki hizalama hedefi + bölme şeridi + numara etiketi.
+       Şerit: x ∈ [-apron_depth + band_width, 0], bölme ekseninde, zemin plakasının
+       üstünde band_height kalınlığında (station_layout.bay_line ile aynı). -->
+  <xacro:property name="bl_x0" value="${-A + V['band_width']}"/>
   <xacro:macro name="bays" params="i">
     <xacro:property name="y" value="${(i - (N - 1) / 2.0) * pitch}"/>
-    <xacro:marker kind="upper" marker_id="${ids[i]}" y="${y}"/>
-    <xacro:marker kind="lower" marker_id="${ids[i] + M['lower_id_offset']}" y="${y}"/>
+    <xacro:box_visual name="bay_line_${ids[i]}" size="${[-bl_x0, V['bay_line']['width'], V['band_height']]}"
+                      xyz="${[bl_x0 / 2.0, y, bt + V['band_height'] / 2.0]}" rgba="${lane_rgba}" cast_shadows="false"/>
     <xacro:align_target bay_id="${ids[i]}" side="right" y="${y - al_off}"/>
     <xacro:align_target bay_id="${ids[i]}" side="left" y="${y + al_off}"/>
