Commit message: feat(cv): F3 + F4 — mission manager, GUI Manual/Auto mode, IMU, drop and transit
F3 (approach + pick, GUI mode):
- forklift_autonomy: ROS-free core (SE2, bay tracker in odom, motion primitives,
  bay-axis servo, mission state machine) and mission_manager node (D-68)
- GUI Manual/Auto panel: IAutonomyPort, AutonomyController, ROS and mock adapters,
  AutonomyPanel.qml, tests (D-69)
- IMU on the robot, attitude from accelerometer + gyro with motion gate and
  median level calibration (D-67)
- A1 acceptance (mission_acceptance --test a1)

F4 (drop + transit):
- one state machine for pick/drop/transit/full (D-74)
- bay selection waits for a stable observation; evidence-based "empty";
  REPOSITION recovery when a bay's bullseye pair is not detected (D-71)
- transit by station sign with PRE_DOCK refinement from bullseye pairs (D-72)
- transit by floor lane with candidate association and short-memory line;
  neutral station's lane is yellow (D-73)
- perception nodes survive a bad frame; NaN Jacobian in the sign pose fit (D-75)
- A2/A3 acceptance; test harness fixes (parking spots, 5 tau after teleport)

Results (sigma = 0, both worlds): A1 36/36, A2 36/36, A3 18/18; unit tests 35/35,
GUI 164/164, S 6/6, T 13/13 (T2 not run, see REPORT_CV §F4.6).

Co-Authored-By: Claude Opus 5.5 <noreply@anthropic.com>

File: docs/logs/T1_forklift_use_sim_false.urdf (robot description, URDF)
Before this commit: robot forklift, 14 links, 13 joints
Links:
- added link imu_link
- link chassis_link: geometry collision box size=0.4 0.3 0.15; visual box size=0.015000000000000013 0.26 0.035
- link left_wheel_link: geometry collision sphere radius=0.05; visual cylinder length=0.03 radius=0.05
- link mast_link: geometry collision box size=0.03 0.03 0.5; collision box size=0.03 0.03 0.5
- link right_wheel_link: geometry collision sphere radius=0.05; visual cylinder length=0.03 radius=0.05
Joints:
- added joint imu_joint: type fixed, parent base_link, child imu_link, origin xyz=-0.12 0.0 0.05 rpy=0 0 0

File: docs/logs/T1_forklift_use_sim_true.urdf (robot description, URDF)
Before this commit: robot forklift, 14 links, 13 joints
Links:
- added link imu_link
- link chassis_link: geometry collision box size=0.4 0.3 0.15; visual box size=0.015000000000000013 0.26 0.035
- link left_wheel_link: geometry collision sphere radius=0.05; visual cylinder length=0.03 radius=0.05
- link mast_link: geometry collision box size=0.03 0.03 0.5; collision box size=0.03 0.03 0.5
- link right_wheel_link: geometry collision sphere radius=0.05; visual cylinder length=0.03 radius=0.05
Joints:
- added joint imu_joint: type fixed, parent base_link, child imu_link, origin xyz=-0.12 0.0 0.05 rpy=0 0 0

File: src/forklift_description/urdf/forklift.urdf.xacro (robot description, xacro)
@@ -27,4 +27,5 @@
   <xacro:include filename="components/fork_carriage.xacro"/>
   <xacro:include filename="components/camera.xacro"/>
+  <xacro:include filename="components/imu.xacro"/>
   <xacro:include filename="components/appearance.xacro"/>
   <!-- gövde ve yürüyüş -->
@@ -39,4 +40,5 @@
   <xacro:mast_camera prefix="${prefix}" name="front_camera" cfg="${cfg}"/>
   <xacro:mast_camera prefix="${prefix}" name="lane_camera" cfg="${cfg}"/>
+  <xacro:imu_frame prefix="${prefix}" cfg="${cfg}"/>
   <!-- yalnızca simülasyon: plugin'ler, sürtünme, sensör blokları -->
   <xacro:if value="$(arg use_sim)">

File: src/forklift_description/urdf/gazebo/forklift.gazebo.xacro (robot description, xacro)
@@ -5,5 +5,5 @@
   yalnızca use_sim:=true iken dahil eder. Üç bağımsız bölüm:
     1) Yüzey      : sürtünme katsayıları (<gazebo reference> → SDF <surface>)
-    2) Sensörler  : iki kamera sensörü
+    2) Sensörler  : iki kamera sensörü, IMU
     3) Kontrol    : DiffDrive, JointPositionController, JointStatePublisher
                     (gz_ros2_control'e geçişte YALNIZCA bu bölüm değişir)
@@ -55,4 +55,20 @@
     </gazebo>
   </xacro:macro>
+  <!-- IMU ekseni gürültüsü (x, y, z aynı): gz-sensors ImuSensor.cc / sdformat <noise> -->
+  <xacro:macro name="imu_axes" params="n">
+    <xacro:macro name="imu_axis" params="axis">
+      <xacro:element xacro:name="${axis}">
+        <noise type="gaussian">
+          <mean>0</mean>
+          <stddev>${n.stddev}</stddev>
+          <bias_mean>${n.bias_mean}</bias_mean>
+          <bias_stddev>${n.bias_stddev}</bias_stddev>
+        </noise>
+      </xacro:element>
+    </xacro:macro>
+    <xacro:imu_axis axis="x"/>
+    <xacro:imu_axis axis="y"/>
+    <xacro:imu_axis axis="z"/>
+  </xacro:macro>
   <xacro:macro name="forklift_gazebo" params="prefix cfg">
     <xacro:property name="gzc" value="${cfg.gazebo}"/>
@@ -69,4 +85,21 @@
     <xacro:gz_camera_sensor prefix="${prefix}" name="front_camera" cam="${cfg.cameras.front_camera}"/>
     <xacro:gz_camera_sensor prefix="${prefix}" name="lane_camera" cam="${cfg.cameras.lane_camera}"/>
+    <!-- IMU (D-67): ivme ve açısal hız, gürültülü; gz-sim-imu-system aşağıda -->
+    <xacro:property name="imu" value="${cfg.imu}"/>
+    <gazebo reference="${prefix}imu_link">
+      <sensor name="imu" type="imu">
+        <always_on>true</always_on>
+        <update_rate>${imu.update_rate}</update_rate>
+        <topic>${imu.topic}</topic>
+        <imu>
+          <angular_velocity>
+            <xacro:imu_axes n="${imu.noise.gyro}"/>
+          </angular_velocity>
+          <linear_acceleration>
+            <xacro:imu_axes n="${imu.noise.accel}"/>
+          </linear_acceleration>
+        </imu>
+      </sensor>
+    </gazebo>
     <!-- ============================ 3) Kontrol ========================== -->
     <gazebo>
@@ -116,4 +149,7 @@
         </xacro:unless>
       </plugin>
+      <!-- IMU sensörlerini güncelleyen sistem (dünyaya değil robota eklenir; robot kendi
+           sensörünü getirir) -->
+      <plugin filename="gz-sim-imu-system" name="gz::sim::systems::Imu"/>
       <!-- Tüm eklemlerin durumu (joint_name verilmediğinde hepsi yayınlanır) -->
       <plugin filename="gz-sim-joint-state-publisher-system"
